Commit message: [feat] 更新BSRL模型并切换为URDF加载

File: source/BSRL_Low_Limb_PPO/BSRL_Low_Limb_PPO/assets/BSRL/bsrl/urdf/export.urdf (robot description, URDF)
Before this commit: robot export, 13 links, 12 joints
Links:
- link base_link: geometry collision box size=0.10 0.10 0.08; collision box size=0.12 0.30 0.035
- link link_left_ankle_pitch: geometry collision cylinder length=0.012 radius=0.025; visual mesh filename=../meshes/link_left_ankle_pitch.obj
- link link_left_ankle_roll: geometry collision cylinder length=0.035 radius=0.025; collision mesh filename=../meshes/left_heel_collision_flat.obj
- link link_left_hip_roll: geometry collision sphere radius=0.04; visual mesh filename=../meshes/link_left_hip_roll.obj
- link link_left_hip_yaw: geometry collision sphere radius=0.04; visual mesh filename=../meshes/link_left_hip_yaw.obj
- link link_left_shank: geometry collision cylinder length=0.2531 radius=0.025; visual mesh filename=../meshes/link_left_shank.obj
- link link_left_thigh: geometry collision cylinder length=0.106 radius=0.035; collision cylinder length=0.16 radius=0.04
- link link_right_ankle_pitch: geometry collision cylinder length=0.012 radius=0.025; visual mesh filename=../meshes/link_right_ankle_pitch.obj
- link link_right_ankle_roll: geometry collision cylinder length=0.035 radius=0.025; collision mesh filename=../meshes/right_heel_collision_flat.obj
- link link_right_hip_roll: geometry collision sphere radius=0.04; visual mesh filename=../meshes/link_right_hip_roll.obj
- link link_right_hip_yaw: geometry collision sphere radius=0.04; visual mesh filename=../meshes/link_right_hip_yaw.obj
- link link_right_shank: geometry collision cylinder length=0.2532 radius=0.025; visual mesh filename=../meshes/link_right_shank.obj
- link link_right_thigh: geometry collision cylinder length=0.106 radius=0.035; collision cylinder length=0.16 radius=0.04
Joints:
- joint joint_left_ankle_pitch: limit lower=-0.6 upper=0.6 effort=1000 velocity=10 -> lower=-0.6 upper=0.6 effort=112 velocity=26.1799
- joint joint_left_ankle_roll: limit lower=-0.52 upper=0.52 effort=1000 velocity=10 -> lower=-0.52 upper=0.52 effort=112 velocity=26.1799
- joint joint_left_hip_pitch: limit lower=-1.5 upper=0.3 effort=1000 velocity=10 -> lower=-1.5 upper=0.3 effort=216 velocity=15.1320
- joint joint_left_hip_roll: limit lower=-0.15 upper=0.15 effort=1000 velocity=10 -> lower=-0.3 upper=0.3 effort=216 velocity=15.1320
- joint joint_left_hip_yaw: limit lower=-0.6 upper=0.4 effort=1000 velocity=10 -> lower=-0.6 upper=0.4 effort=112 velocity=26.1799
- joint joint_left_knee_pitch: limit lower=0 upper=2.2 effort=1000 velocity=10 -> lower=-0.1 upper=2.2 effort=216 velocity=15.1320
- joint joint_right_ankle_pitch: limit lower=-0.6 upper=0.6 effort=1000 velocity=10 -> lower=-0.6 upper=0.6 effort=112 velocity=26.1799
- joint joint_right_ankle_roll: limit lower=-0.52 upper=0.52 effort=1000 velocity=10 -> lower=-0.52 upper=0.52 effort=112 velocity=26.1799
- joint joint_right_hip_pitch: limit lower=-1.5 upper=0.3 effort=1000 velocity=10 -> lower=-1.5 upper=0.3 effort=216 velocity=15.1320
- joint joint_right_hip_roll: limit lower=-0.15 upper=0.15 effort=1000 velocity=10 -> lower=-0.3 upper=0.3 effort=216 velocity=15.1320
- joint joint_right_hip_yaw: limit lower=-0.4 upper=0.6 effort=1000 velocity=10 -> lower=-0.4 upper=0.6 effort=112 velocity=26.1799
- joint joint_right_knee_pitch: limit lower=0 upper=2.2 effort=1000 velocity=10 -> lower=-0.1 upper=2.2 effort=216 velocity=15.1320

File: source/BSRL_Low_Limb_PPO/BSRL_Low_Limb_PPO/assets/BSRL/bsrl/urdf/export_floating.urdf (robot description, URDF)
Before this commit: robot export_floating, 14 links, 13 joints
Links:
- link base_link: geometry collision box size=0.10 0.10 0.08; collision box size=0.12 0.30 0.035
- link link_left_ankle_pitch: geometry collision cylinder length=0.012 radius=0.025; visual mesh filename=../meshes/link_left_ankle_pitch.obj
- link link_left_ankle_roll: geometry collision cylinder length=0.035 radius=0.025; collision mesh filename=../meshes/left_heel_collision_flat.obj
- link link_left_hip_roll: geometry collision sphere radius=0.04; visual mesh filename=../meshes/link_left_hip_roll.obj
- link link_left_hip_yaw: geometry collision sphere radius=0.04; visual mesh filename=../meshes/link_left_hip_yaw.obj
- link link_left_shank: geometry collision cylinder length=0.2531 radius=0.025; visual mesh filename=../meshes/link_left_shank.obj
- link link_left_thigh: geometry collision cylinder length=0.106 radius=0.035; collision cylinder length=0.16 radius=0.04
- link link_right_ankle_pitch: geometry collision cylinder length=0.012 radius=0.025; visual mesh filename=../meshes/link_right_ankle_pitch.obj
- link link_right_ankle_roll: geometry collision cylinder length=0.035 radius=0.025; collision mesh filename=../meshes/right_heel_collision_flat.obj
- link link_right_hip_roll: geometry collision sphere radius=0.04; visual mesh filename=../meshes/link_right_hip_roll.obj
- link link_right_hip_yaw: geometry collision sphere radius=0.04; visual mesh filename=../meshes/link_right_hip_yaw.obj
- link link_right_shank: geometry collision cylinder length=0.2532 radius=0.025; visual mesh filename=../meshes/link_right_shank.obj
- link link_right_thigh: geometry collision cylinder length=0.106 radius=0.035; collision cylinder length=0.16 radius=0.04
Joints:
- joint joint_left_ankle_pitch: limit lower=-0.6 upper=0.6 effort=1000 velocity=10 -> lower=-0.6 upper=0.6 effort=112 velocity=26.1799
- joint joint_left_ankle_roll: limit lower=-0.52 upper=0.52 effort=1000 velocity=10 -> lower=-0.52 upper=0.52 effort=112 velocity=26.1799
- joint joint_left_hip_pitch: limit lower=-1.5 upper=0.3 effort=1000 velocity=10 -> lower=-1.5 upper=0.3 effort=216 velocity=15.1320
- joint joint_left_hip_roll: limit lower=-0.15 upper=0.15 effort=1000 velocity=10 -> lower=-0.3 upper=0.3 effort=216 velocity=15.1320
- joint joint_left_hip_yaw: limit lower=-0.6 upper=0.4 effort=1000 velocity=10 -> lower=-0.6 upper=0.4 effort=112 velocity=26.1799
- joint joint_left_knee_pitch: limit lower=0 upper=2.2 effort=1000 velocity=10 -> lower=-0.1 upper=2.2 effort=216 velocity=15.1320
- joint joint_right_ankle_pitch: limit lower=-0.6 upper=0.6 effort=1000 velocity=10 -> lower=-0.6 upper=0.6 effort=112 velocity=26.1799
- joint joint_right_ankle_roll: limit lower=-0.52 upper=0.52 effort=1000 velocity=10 -> lower=-0.52 upper=0.52 effort=112 velocity=26.1799
- joint joint_right_hip_pitch: limit lower=-1.5 upper=0.3 effort=1000 velocity=10 -> lower=-1.5 upper=0.3 effort=216 velocity=15.1320
- joint joint_right_hip_roll: limit lower=-0.15 upper=0.15 effort=1000 velocity=10 -> lower=-0.3 upper=0.3 effort=216 velocity=15.1320
- joint joint_right_hip_yaw: limit lower=-0.4 upper=0.6 effort=1000 velocity=10 -> lower=-0.4 upper=0.6 effort=112 velocity=26.1799
- joint joint_right_knee_pitch: limit lower=0 upper=2.2 effort=1000 velocity=10 -> lower=-0.1 upper=2.2 effort=216 velocity=15.1320
